File: I2C-Codeline-Matrix.brd (EAGLE design)
At the start: 86.5 x 100 mm, 12 parts, among them CON1 CONNECTOR-I2CLEFT, CON2 CONNECTOR-I2CLEFT, CON3 CONNECTOR-GROVE-4P-2.0-347013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, CON4 CONNECTOR-GROVE-4P-2.0-347013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

Commit message: 2.1
Parts:
- moved CON4 10.5 mm to (73.7, 36.8)
- moved CON1 8.03 mm to (73.7, 26.7)
- moved CON3 7.73 mm to (7.62, 36.8)
- moved CON2 7.73 mm to (7.62, 26.7)
- moved JP1 1.27 mm to (22.9, 45.7)
- moved JP2 1.27 mm to (20.3, 45.7)
- moved JP3 1.27 mm to (17.8, 45.7)
Connections:
- net GND: now also MATRIX2.G@2
- net VCCIO: now also MATRIX2.V+@2
Routing:
- net N$1: track 158.0 -> 73.6 mm
- net SDA: track 140.6 -> 149.2 mm
- net GND: track 0.00 -> 7.24 mm
- net SCL: track 127.0 -> 132.3 mm
- net N$8: track 42.6 -> 41.3 mm
- net N$7: track 39.0 -> 37.7 mm
- net N$6: track 35.4 -> 34.1 mm
Other:
- board text added: "2019.02"
- board text added: "Codeline Display"
- board text added: "I2C LED Matrix"
- board text added: "v2.1"
- board text removed: "2018.12"
- board text removed: "I2C Display Board"
- board text removed: "v2.0"

Commit message: added values for connectors
Parts:
- JP1, JP2, JP3: value (none) -> 0.100
Changed lines of the file:
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@@
 <attribute name="VALUE" x="84.455" y="31.115" size="0.635" layer="27" font="vector" ratio="10" rot="R90"/>
 </element>
-<element name="JP1" library="SPCoast" package="1X02_LOCK" value="" x="22.86" y="45.72" rot="R270"/>
-<element name="JP2" library="SPCoast" package="1X02_LOCK" value="" x="20.32" y="45.72" rot="R270"/>
-<element name="JP3" library="SPCoast" package="1X02_LOCK" value="" x="17.78" y="45.72" rot="R270"/>
+<element name="JP1" library="SPCoast" package="1X02_LOCK" value="0.100" x="22.86" y="45.72" rot="R270"/>
+<element name="JP2" library="SPCoast" package="1X02_LOCK" value="0.100" x="20.32" y="45.72" rot="R270"/>
+<element name="JP3" library="SPCoast" package="1X02_LOCK" value="0.100" x="17.78" y="45.72" rot="R270"/>
 </elements>
 <signals>

Commit message: normalized values
Parts:
- ARDUINO1: value ARDUINO-PRO-MINIDAVESROBOT -> DAVEK
- BOARD: value BOARD80X150 -> BOARD
- CON1, CON2: value CONNECTOR-I2CLEFT -> I2C
- CON3, CON4: value CONNECTOR-GROVE-4P-2.0-3470130P1 -> 2mm
- MATRIX1, MATRIX2: value LEDMATRIX -> 8x8
- OSHW1: value OSHW-LOGOL -> OSHW
Changed lines of the file:
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@@
 </autorouter>
 <elements>
-<element name="OSHW1" library="SparkFun" package="OSHW-LOGO-L" value="OSHW-LOGOL" x="22.86" y="33.02" smashed="yes"/>
-<element name="BOARD" library="SPCoast" package="BOARD-DINRAIL-3.17INX8CM-NOHOLES" value="BOARD80X150" x="0" y="0" smashed="yes"/>
-<element name="MATRIX1" library="SPCoast" package="LEDMATRIX" value="LEDMATRIX" x="45.72" y="68.58" smashed="yes">
+<element name="OSHW1" library="SparkFun" package="OSHW-LOGO-L" value="OSHW" x="22.86" y="33.02" smashed="yes"/>
+<element name="BOARD" library="SPCoast" package="BOARD-DINRAIL-3.17INX8CM-NOHOLES" value="BOARD" x="0" y="0" smashed="yes"/>
+<element name="MATRIX1" library="SPCoast" package="LEDMATRIX" value="8x8" x="45.72" y="68.58" smashed="yes">
 <attribute name="NAME" x="27.94" y="52.07" size="1.27" layer="25" font="vector" rot="R90"/>
 </element>
-<element name="MATRIX2" library="SPCoast" package="LEDMATRIX" value="LEDMATRIX" x="45.72" y="31.75" smashed="yes">
+<element name="MATRIX2" library="SPCoast" package="LEDMATRIX" value="8x8" x="45.72" y="31.75" smashed="yes">
 <attribute name="NAME" x="27.94" y="15.24" size="1.27" layer="25" font="vector" rot="R90"/>
 </element>
-<element name="ARDUINO1" library="SPCoast" package="ARDUINO_PRO_MINI_DAVEK" value="ARDUINO-PRO-MINIDAVESROBOT" x="26.67" y="88.9" rot="R180"/>
-<element name="CON1" library="SPCoast" package="I2C-L" value="CONNECTOR-I2CLEFT" x="73.66" y="26.67" smashed="yes">
+<element name="ARDUINO1" library="SPCoast" package="ARDUINO_PRO_MINI_DAVEK" value="DAVEK" x="26.67" y="88.9" rot="R180"/>
+<element name="CON1" library="SPCoast" package="I2C-L" value="I2C" x="73.66" y="26.67" smashed="yes">
 <attribute name="NAME" x="84.328" y="25.654" size="0.889" layer="25" font="vector" ratio="11" rot="R90"/>
 <attribute name="VALUE" x="84.328" y="13.589" size="0.635" layer="27" font="vector" ratio="10" rot="R90"/>
 </element>
-<element name="CON2" library="SPCoast" package="I2C-L" value="CONNECTOR-I2CLEFT" x="7.62" y="26.67" smashed="yes">
+<element name="CON2" library="SPCoast" package="I2C-L" value="I2C" x="7.62" y="26.67" smashed="yes">
 <attribute name="NAME" x="-3.302" y="12.954" size="0.889" layer="25" font="vector" ratio="11" rot="R90"/>
 <attribute name="VALUE" x="-3.302" y="19.939" size="0.635" layer="27" font="vector" ratio="10" rot="R90"/>
 </element>
-<element name="CON3" library="SPCoast" package="4P-2.0" value="CONNECTOR-GROVE-4P-2.0-3470130P1" x="7.62" y="36.83" smashed="yes" rot="R90">
+<element name="CON3" library="SPCoast" package="4P-2.0" value="2mm" x="7.62" y="36.83" smashed="yes" rot="R90">
 <attribute name="NAME" x="-2.54" y="34.925" size="0.889" layer="25" font="vector" ratio="11" rot="R90"/>
 <attribute name="VALUE" x="9.525" y="34.925" size="0.635" layer="27" font="vector" ratio="10" rot="R90"/>
 </element>
-<element name="CON4" library="SPCoast" package="4P-2.0" value="CONNECTOR-GROVE-4P-2.0-3470130P1" x="73.66" y="36.83" smashed="yes" rot="R90">
+<element name="CON4" library="SPCoast" package="4P-2.0" value="2mm" x="73.66" y="36.83" smashed="yes" rot="R90">
 <attribute name="NAME" x="86.36" y="34.925" size="0.889" layer="25" font="vector" ratio="11" rot="R90"/>
 <attribute name="VALUE" x="84.455" y="31.115" size="0.635" layer="27" font="vector" ratio="10" rot="R90"/>
